File: green_house_controller.kicad_pcb (KiCad board)
At the start: 2 copper layers, 104.9 x 76.2 mm, 111 parts, among them J1 TC2030-IDC, J2 Screw_Terminal_01x10, J3 USB_B_Mini, J4 Screw_Terminal_01x06, J5 Screw_Terminal_01x03, J6 Barrel_Jack, Q1 2N7002, Q10 DMG3406L, Q11 DMP3068L, Q12 DMG3406L, Q13 2N7002, Q14 DMP3068L, Q15 DMG3406L, Q16 DMP3068L, Q17 DMG3406L, Q19 2N7002, Q2 2N7002, Q3 DMP3068L, Q4 DMG3406L, Q5 DMP3068L, Q6 DMG3406L, Q7 2N7002, Q8 2N7002, Q9 DMP3068L, SW1 SW_Push, U1 ESP32-WROVER, U2 TPS54231, U3 TLP3825TP1_F, U4 TLP3825TP1_F, U5 TLP3825TP1_F, U6 TLP3825TP1_F, U7 LM2733XMF, U8 DHT11

Commit message: Replaced relays with smd versions.
Parts:
- C2: value 20uF -> 10uF
- U3, U4, U5, U6: footprint Package_DIP:DIP-8_W7.62mm -> Package_DIP:DIP-8_W7.62mm_SMDSocket_SmallPads
- moved U6 5.56 mm to (184.3, 118.0)
- moved U5 5.10 mm to (173.5, 118.0)
- moved U3 4.68 mm to (162.7, 118.0)
- moved U4 4.32 mm to (151.9, 118.0)
Routing:
- net GND: track 136.6 -> 107.2 mm, vias 61 -> 62
- net /microcontroller/FAN_1_CTRL: track 51.0 -> 49.6 mm
- net Net-(R21-Pad1): track 10.9 -> 12.3 mm
- net Net-(R20-Pad1): track 11.8 -> 12.9 mm, vias 1 -> 2
- net Net-(R23-Pad1): track 12.6 -> 13.2 mm, vias 1 -> 2
- net Net-(R22-Pad1): track 12.7 -> 13.1 mm, vias 1 -> 2
- net /relay control/110VAC: vias 0 -> 8
- added copper zone on F.Cu, net /relay control/110VAC
